Commit message: Gazebo Files

File: description/xacro/rrr_arm.urdf.xacro (robot description, xacro)
@@ -1,5 +1,5 @@
 <?xml version="1.0"?>
 <!-- Make the namespace of the robot-->
-<robot name="rrr_arm" xmlns:xacro="http://www.ros.org/wiki/xacro">
+<robot xmlns:xacro="http://www.ros.org/wiki/xacro" name="rrr_arm">
     <!--Define constants-->
     <xacro:property name="link_type" value="cuboidal" />
@@ -23,5 +23,5 @@
     <xacro:property name="length_5" value="0.15" /> <!--gripper base length-->
     <xacro:property name="length_6" value="0.07" /> <!--finger length-->
-    <!--Define colors-->
+    <!--Define Rviz colors-->
     <material name="Black">
         <color rgba="0.0 0.0 0.0 1.0"/>
@@ -53,7 +53,51 @@
     </inertial>
     </xacro:macro>
-    <!--=============================================================================-->
+    <!-- macros for transmission -->
+    <xacro:macro name="transmission_block" params="joint_name">
+	  <transmission name="tran1">
+	    <type>transmission_interface/SimpleTransmission</type>
+	    <joint name="${joint_name}">
+	      <hardwareInterface>hardware_interface/PositionJointInterface</hardwareInterface>
+	    </joint>
+	    <actuator name="motor1">
+	      <hardwareInterface>hardware_interface/PositionJointInterface</hardwareInterface>
+	      <mechanicalReduction>1</mechanicalReduction>
+	    </actuator>
+	  </transmission>
+   </xacro:macro>
+    <!--Define Gazebo colors-->
+    <xacro:macro name="gazebo_grey_link_color_block" params="link_name">
+    <gazebo reference="${link_name}">
+    <visual>
+      <material>
+        <ambient>0.5 0.5 0.5 1.0</ambient>
+        <diffuse>0.56666695 0.56666695 0.56666695 1.0</diffuse>
+        <specular>0.6000003 0.6000003 0.6000003 1.0</specular>
+      </material>
+    </visual>
+    </gazebo>
+  </xacro:macro>
+  <xacro:macro name="gazebo_blue_link_color_block" params="link_name">
+    <gazebo reference="${link_name}">
+    <visual>
+      <material>
+        <ambient>0.589 0.793 1.0 1.0</ambient>
+        <diffuse>0.56666695 0.56666695 0.56666695 1.0</diffuse>
+        <specular>0.6000003 0.6000003 0.6000003 1.0</specular>
+      </material>
+    </visual>
+    </gazebo>
+  </xacro:macro>
+    <!--=============================================================================-->
+    <!--world link-->
+    <link name="world"/>
+    <joint name="world_joint" type="fixed">
+        <origin xyz="0.0 0.0 0.0" rpy="0.0 0.0 0.0"/>
+        <parent link="world"/>
+        <child link="base_link"/>
+    </joint>
     <!--base_link-->
     <link name="base_link">
+        <xacro:inertial_block mass="${mass_1}" length="${length_1}" radius="${radius_1}"/>
         <visual>
             <origin xyz="0.0 0.0 ${length_1/2.0}" rpy="0.0 0.0 0.0"/>
@@ -70,4 +114,5 @@
         </collision>
     </link>
+    <xacro:gazebo_blue_link_color_block link_name="base_link"/>
     <joint name="joint_1" type="revolute">
         <origin xyz="0.0 0.0 ${length_1}" rpy="0.0 0.0 0.0"/>
@@ -95,4 +140,6 @@
         </collision>
     </link>
+    <xacro:gazebo_grey_link_color_block link_name="link_1"/>
+    <!-- <xacro:gazebo_grey_link_color_block link_name="link_1"> -->
     <link name="link_1_endlink">
         <xacro:inertial_block mass="${mass_2/3.0}" length="${2*radius_2+2*radius_3}" radius="${radius_2}"/>
@@ -111,4 +158,5 @@
         </collision>
     </link>
+    <xacro:gazebo_blue_link_color_block link_name="link_1_endlink"/>
     <joint name="link_1_endjoint" type="fixed">
         <origin xyz="${-radius_2} 0.0 ${length_2 - 0.01}" rpy="0.0 ${M_PI/2.0} 0.0"/>
@@ -116,4 +164,8 @@
         <child link="link_1_endlink"/>
     </joint>
+    <gazebo reference="link_1_endjoint">
+        <disableFixedJointLumping>true</disableFixedJointLumping>
+        <preserveFixedJoint>true</preserveFixedJoint>
+    </gazebo>
     <joint name="joint_2" type="revolute">
         <origin xyz="${radius_2 + radius_3} 0.0 ${length_2}" rpy="0.0 0.0 0.0"/>
@@ -138,7 +190,8 @@
             <geometry>
                 <cylinder radius="${radius_3}" length="${length_3}"/>
-            </geometry>>
-        </collision>
-    </link>
+            </geometry>
+        </collision>
+    </link>
+    <xacro:gazebo_grey_link_color_block link_name="link_2"/>
     <link name="link_2_endlink">
         <xacro:inertial_block mass="${mass_3/3.0}" length="${2*radius_3+2*radius_4}" radius="${radius_3}"/>
@@ -157,4 +210,5 @@
         </collision>
     </link>
+    <xacro:gazebo_blue_link_color_block link_name="link_2_endlink"/>
     <joint name="link_2_endjoint" type="fixed">
         <origin xyz="${-radius_3} 0.0 ${length_3 - 0.01}" rpy="0.0 ${M_PI/2.0} 0.0"/>
@@ -162,4 +216,8 @@
         <child link="link_2_endlink"/>
     </joint>
+    <gazebo reference="link_2_endjoint">
+        <disableFixedJointLumping>true</disableFixedJointLumping>
+        <preserveFixedJoint>true</preserveFixedJoint>
+    </gazebo>
     <joint name="joint_3" type="revolute">
         <origin xyz="${radius_3 + radius_4} 0.0 ${length_3 - radius_3}" rpy="0.0 0.0 0.0"/>
@@ -184,7 +242,8 @@
             <geometry>
                 <cylinder radius="${radius_4}" length="${length_4}"/>
-            </geometry>>
-        </collision>
-    </link>
+            </geometry>
+        </collision>
+    </link>
+    <xacro:gazebo_grey_link_color_block link_name="link_3"/>
     <joint name="joint_4" type="fixed">
         <origin xyz="0.0 0.0 ${length_4}" rpy="0.0 0.0 0.0"/>
@@ -209,7 +268,8 @@
             <geometry>
                 <box size="${radius_5*2} ${radius_5*2} ${length_5}"/>
-            </geometry>>
-        </collision>
-    </link>
+            </geometry>
+        </collision>
+    </link>
+    <xacro:gazebo_grey_link_color_block link_name="link_4"/>
     <joint name="gripper_joint_1" type="prismatic">
         <origin xyz="0.0 0.0 ${radius_5 + length_6/2.0}" rpy="0.0 0.0 0.0"/>
@@ -246,7 +306,8 @@
             <geometry>
                 <box size="${radius_6*2} ${radius_6*2} ${length_6}"/>
-            </geometry>>
-        </collision>
-    </link>
+            </geometry>
+        </collision>
+    </link>
+    <xacro:gazebo_grey_link_color_block link_name="gripper_link_1"/>
     <!--=============================================================================-->
     <!--gripper_link_2-->
@@ -267,4 +328,5 @@
         </collision>
     </link>
+    <xacro:gazebo_grey_link_color_block link_name="gripper_link_2"/>
     <!--=============================================================================-->
     <!--gripper_frame_cp-->
@@ -285,3 +347,16 @@
         </collision>
     </link>
+    <!-- Transmissions for ros control -->
+    <xacro:transmission_block joint_name="joint_1"/>
+    <xacro:transmission_block joint_name="joint_2"/>
+    <xacro:transmission_block joint_name="joint_3"/>
+    <xacro:transmission_block joint_name="joint_4"/>
+    <xacro:transmission_block joint_name="gripper_joint_1"/>
+    <xacro:transmission_block joint_name="gripper_joint_2"/>
+    <!-- ros_control plugin -->
+    <!-- <gazebo>
+        <plugin name="gazebo_ros_control" filename="libgazebo_ros_control.so">
+        <robotNamespace>/rrr_arm</robotNamespace>
+        </plugin>
+    </gazebo> -->
 </robot>

Commit message: Gazebo Files

File: description/xacro/rrr_arm.urdf.xacro (robot description, xacro)
@@ -1,5 +1,5 @@
 <?xml version="1.0"?>
 <!-- Make the namespace of the robot-->
-<robot name="rrr_arm" xmlns:xacro="http://www.ros.org/wiki/xacro">
+<robot xmlns:xacro="http://www.ros.org/wiki/xacro" name="rrr_arm">
     <!--Define constants-->
     <xacro:property name="link_type" value="cuboidal" />
@@ -23,5 +23,5 @@
     <xacro:property name="length_5" value="0.15" /> <!--gripper base length-->
     <xacro:property name="length_6" value="0.07" /> <!--finger length-->
-    <!--Define colors-->
+    <!--Define Rviz colors-->
     <material name="Black">
         <color rgba="0.0 0.0 0.0 1.0"/>
@@ -53,7 +53,51 @@
     </inertial>
     </xacro:macro>
-    <!--=============================================================================-->
+    <!-- macros for transmission -->
+    <xacro:macro name="transmission_block" params="joint_name">
+	  <transmission name="tran1">
+	    <type>transmission_interface/SimpleTransmission</type>
+	    <joint name="${joint_name}">
+	      <hardwareInterface>hardware_interface/PositionJointInterface</hardwareInterface>
+	    </joint>
+	    <actuator name="motor1">
+	      <hardwareInterface>hardware_interface/PositionJointInterface</hardwareInterface>
+	      <mechanicalReduction>1</mechanicalReduction>
+	    </actuator>
+	  </transmission>
+   </xacro:macro>
+    <!--Define Gazebo colors-->
+    <xacro:macro name="gazebo_grey_link_color_block" params="link_name">
+    <gazebo reference="${link_name}">
+    <visual>
+      <material>
+        <ambient>0.5 0.5 0.5 1.0</ambient>
+        <diffuse>0.56666695 0.56666695 0.56666695 1.0</diffuse>
+        <specular>0.6000003 0.6000003 0.6000003 1.0</specular>
+      </material>
+    </visual>
+    </gazebo>
+  </xacro:macro>
+  <xacro:macro name="gazebo_blue_link_color_block" params="link_name">
+    <gazebo reference="${link_name}">
+    <visual>
+      <material>
+        <ambient>0.589 0.793 1.0 1.0</ambient>
+        <diffuse>0.56666695 0.56666695 0.56666695 1.0</diffuse>
+        <specular>0.6000003 0.6000003 0.6000003 1.0</specular>
+      </material>
+    </visual>
+    </gazebo>
+  </xacro:macro>
+    <!--=============================================================================-->
+    <!--world link-->
+    <link name="world"/>
+    <joint name="world_joint" type="fixed">
+        <origin xyz="0.0 0.0 0.0" rpy="0.0 0.0 0.0"/>
+        <parent link="world"/>
+        <child link="base_link"/>
+    </joint>
     <!--base_link-->
     <link name="base_link">
+        <xacro:inertial_block mass="${mass_1}" length="${length_1}" radius="${radius_1}"/>
         <visual>
             <origin xyz="0.0 0.0 ${length_1/2.0}" rpy="0.0 0.0 0.0"/>
@@ -70,4 +114,5 @@
         </collision>
     </link>
+    <xacro:gazebo_blue_link_color_block link_name="base_link"/>
     <joint name="joint_1" type="revolute">
         <origin xyz="0.0 0.0 ${length_1}" rpy="0.0 0.0 0.0"/>
@@ -95,4 +140,6 @@
         </collision>
     </link>
+    <xacro:gazebo_grey_link_color_block link_name="link_1"/>
+    <!-- <xacro:gazebo_grey_link_color_block link_name="link_1"> -->
     <link name="link_1_endlink">
         <xacro:inertial_block mass="${mass_2/3.0}" length="${2*radius_2+2*radius_3}" radius="${radius_2}"/>
@@ -111,4 +158,5 @@
         </collision>
     </link>
+    <xacro:gazebo_blue_link_color_block link_name="link_1_endlink"/>
     <joint name="link_1_endjoint" type="fixed">
         <origin xyz="${-radius_2} 0.0 ${length_2 - 0.01}" rpy="0.0 ${M_PI/2.0} 0.0"/>
@@ -116,4 +164,8 @@
         <child link="link_1_endlink"/>
     </joint>
+    <gazebo reference="link_1_endjoint">
+        <disableFixedJointLumping>true</disableFixedJointLumping>
+        <preserveFixedJoint>true</preserveFixedJoint>
+    </gazebo>
     <joint name="joint_2" type="revolute">
         <origin xyz="${radius_2 + radius_3} 0.0 ${length_2}" rpy="0.0 0.0 0.0"/>
@@ -141,4 +193,5 @@
         </collision>
     </link>
+    <xacro:gazebo_grey_link_color_block link_name="link_2"/>
     <link name="link_2_endlink">
         <xacro:inertial_block mass="${mass_3/3.0}" length="${2*radius_3+2*radius_4}" radius="${radius_3}"/>
@@ -157,4 +210,5 @@
         </collision>
     </link>
+    <xacro:gazebo_blue_link_color_block link_name="link_2_endlink"/>
     <joint name="link_2_endjoint" type="fixed">
         <origin xyz="${-radius_3} 0.0 ${length_3 - 0.01}" rpy="0.0 ${M_PI/2.0} 0.0"/>
@@ -162,4 +216,8 @@
         <child link="link_2_endlink"/>
     </joint>
+    <gazebo reference="link_2_endjoint">
+        <disableFixedJointLumping>true</disableFixedJointLumping>
+        <preserveFixedJoint>true</preserveFixedJoint>
+    </gazebo>
     <joint name="joint_3" type="revolute">
         <origin xyz="${radius_3 + radius_4} 0.0 ${length_3 - radius_3}" rpy="0.0 0.0 0.0"/>
@@ -187,4 +245,5 @@
         </collision>
     </link>
+    <xacro:gazebo_grey_link_color_block link_name="link_3"/>
     <joint name="joint_4" type="fixed">
         <origin xyz="0.0 0.0 ${length_4}" rpy="0.0 0.0 0.0"/>
@@ -212,4 +271,5 @@
         </collision>
     </link>
+    <xacro:gazebo_grey_link_color_block link_name="link_4"/>
     <joint name="gripper_joint_1" type="prismatic">
         <origin xyz="0.0 0.0 ${radius_5 + length_6/2.0}" rpy="0.0 0.0 0.0"/>
@@ -249,4 +309,5 @@
         </collision>
     </link>
+    <xacro:gazebo_grey_link_color_block link_name="gripper_link_1"/>
     <!--=============================================================================-->
     <!--gripper_link_2-->
@@ -267,4 +328,5 @@
         </collision>
     </link>
+    <xacro:gazebo_grey_link_color_block link_name="gripper_link_2"/>
     <!--=============================================================================-->
     <!--gripper_frame_cp-->
@@ -285,3 +347,16 @@
         </collision>
     </link>
+    <!-- Transmissions for ros control -->
+    <xacro:transmission_block joint_name="joint_1"/>
+    <xacro:transmission_block joint_name="joint_2"/>
+    <xacro:transmission_block joint_name="joint_3"/>
+    <xacro:transmission_block joint_name="joint_4"/>
+    <xacro:transmission_block joint_name="gripper_joint_1"/>
+    <xacro:transmission_block joint_name="gripper_joint_2"/>
+    <!-- ros_control plugin -->
+    <!-- <gazebo>
+        <plugin name="gazebo_ros_control" filename="libgazebo_ros_control.so">
+        <robotNamespace>/rrr_arm</robotNamespace>
+        </plugin>
+    </gazebo> -->
 </robot>
